Commit message: Contains urdf files of the bot, sensors

File: src/line_follower_bot/urdf/properties.xacro (robot description, xacro)
@@ -12,4 +12,9 @@
     <xacro:property name="camera_offset_y" value="0" />
     <xacro:property name="camera_offset_z" value="0.1" />
+    <xacro:property name="lidar_radius" value="0.05" />
+    <xacro:property name="lidar_length" value="0.08" />
+    <xacro:property name="lidar_offset_x" value="0" />
+    <xacro:property name="lidar_offset_y" value="0" />
+    <xacro:property name="lidar_offset_z" value="0.16" />
     <material name="black">
         <color rgba="0 0 0 1" />
